File: learn_to_solder/learn_to_solder.kicad_sch (KiCad schematic)
At the start: 8 parts, among them Q1 2N3904

Commit message: Updated readme and silkscreen
Updated readme to correctly reflect kit components. Added labels in front silkscreen with resistor values to make assembly easier. Rearranged resistors to put both 220s next to each other.
Parts:
- R1: value R -> 47K
- R3, R4: value R -> 220
Changed lines of the file:
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@@
       (effects (font (size 1.27 1.27)) (justify left))
     )
-    (property "Value" "R" (id 1) (at 87.63 107.9499 0)
+    (property "Value" "220" (id 1) (at 87.63 107.9499 0)
       (effects (font (size 1.27 1.27)) (justify left))
     )
@@
       (effects (font (size 1.27 1.27)) (justify left))
     )
-    (property "Value" "R" (id 1) (at 97.79 107.9499 0)
+    (property "Value" "220" (id 1) (at 97.79 107.9499 0)
       (effects (font (size 1.27 1.27)) (justify left))
     )
@@
       (effects (font (size 1.27 1.27)) (justify left))
     )
-    (property "Value" "R" (id 1) (at 68.58 100.3299 0)
+    (property "Value" "47K" (id 1) (at 68.58 100.3299 0)
       (effects (font (size 1.27 1.27)) (justify left))
     )
@@
     )
     (path "/550a9c6f-df40-4a1c-9e90-c0271619fe3c"
-      (reference "R1") (unit 1) (value "R") (footprint "Resistor_THT:R_Axial_DIN0207_L6.3mm_D2.5mm_P10.16mm_Horizontal")
+      (reference "R1") (unit 1) (value "47K") (footprint "Resistor_THT:R_Axial_DIN0207_L6.3mm_D2.5mm_P10.16mm_Horizontal")
     )
     (path "/2aee96ed-5783-466b-9d5f-a794a1219ac4"
@@
     )
     (path "/2f4b6104-fb6f-4667-a51c-8d1090aab2e9"
-      (reference "R3") (unit 1) (value "R") (footprint "Resistor_THT:R_Axial_DIN0207_L6.3mm_D2.5mm_P10.16mm_Horizontal")
+      (reference "R3") (unit 1) (value "220") (footprint "Resistor_THT:R_Axial_DIN0207_L6.3mm_D2.5mm_P10.16mm_Horizontal")
     )
     (path "/51513777-ad0b-4ebb-98c0-52fd72a93ce6"
-      (reference "R4") (unit 1) (value "R") (footprint "Resistor_THT:R_Axial_DIN0207_L6.3mm_D2.5mm_P10.16mm_Horizontal")
+      (reference "R4") (unit 1) (value "220") (footprint "Resistor_THT:R_Axial_DIN0207_L6.3mm_D2.5mm_P10.16mm_Horizontal")
     )
   )

Commit message: V2 updates
Rearranged resistors to group both 220s together. Added slide switch to turn off without removing battery. Corrected typos in silkscreen. Fixed clip slot size.
Parts:
- added SW1: SW_SPDT, Button_Switch_THT:SW_Slide_1P2T_CK_OS102011MS2Q, symbol Switch:SW_SPDT
- Q1: footprint Package_TO_SOT_THT:TO-92_Inline -> Package_TO_SOT_THT:TO-92_Inline_Wide
Connections:
- net GND: now also SW1.1 (A); no longer BT1.2 (-)
- new net: BT1.2 (-), SW1.2 (B)
Changed lines of the file:
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@@
     (stroke (width 0) (type default) (color 0 0 0 0))
   )
-  (wire (pts (xy 50.8 105.41) (xy 50.8 113.03))
+  (wire (pts (xy 53.34 125.73) (xy 50.8 125.73))
     (stroke (width 0) (type default) (color 0 0 0 0))
   )
@@
   )
   (wire (pts (xy 85.09 110.49) (xy 85.09 114.3))
+    (stroke (width 0) (type default) (color 0 0 0 0))
+  )
+  (wire (pts (xy 53.34 115.57) (xy 53.34 125.73))
     (stroke (width 0) (type default) (color 0 0 0 0))
   )
@@
     (pin "1")
   )
+  (symbol (lib_id "Switch:SW_SPDT") (at 50.8 110.49 270) (unit 1)
+    (in_bom yes) (on_board yes) (fields_autoplaced)
+    (property "Reference" "SW1" (id 0) (at 54.61 109.2199 90)
+      (effects (font (size 1.27 1.27)) (justify left))
+    )
+    (property "Value" "SW_SPDT" (id 1) (at 54.61 111.7599 90)
+      (effects (font (size 1.27 1.27)) (justify left))
+    )
+    (property "Footprint" "Button_Switch_THT:SW_Slide_1P2T_CK_OS102011MS2Q" (id 2) (at 50.8 110.49 0)
+      (effects (font (size 1.27 1.27)) hide)
+    )
+    (property "Datasheet" "~" (id 3) (at 50.8 110.49 0)
+      (effects (font (size 1.27 1.27)) hide)
+    )
+    (pin "1")
+    (pin "2")
+    (pin "3")
+  )
   (symbol (lib_id "Device:R_Photo") (at 66.04 109.22 0) (unit 1)
     (in_bom yes) (on_board yes) (fields_autoplaced)
@@
   )
   (symbol (lib_id "Transistor_BJT:2N3904") (at 82.55 119.38 0) (unit 1)
-    (in_bom yes) (on_board yes) (fields_autoplaced)
+    (in_bom yes) (on_board yes)
     (property "Reference" "Q1" (id 0) (at 87.63 118.1099 0)
       (effects (font (size 1.27 1.27)) (justify left))
@@
       (effects (font (size 1.27 1.27)) (justify left))
     )
-    (property "Footprint" "Package_TO_SOT_THT:TO-92_Inline" (id 2) (at 87.63 121.285 0)
-      (effects (font (size 1.27 1.27) italic) (justify left) hide)
+    (property "Footprint" "Package_TO_SOT_THT:TO-92_Inline_Wide" (id 2) (at 62.23 147.32 0)
+      (effects (font (size 1.27 1.27) italic) (justify left))
     )
     (property "Datasheet" "https://www.onsemi.com/pub/Collateral/2N3903-D.PDF" (id 3) (at 82.55 119.38 0)
@@
     (pin "2")
   )
-  (symbol (lib_id "power:GND") (at 50.8 113.03 0) (unit 1)
-    (in_bom yes) (on_board yes) (fields_autoplaced)
-    (property "Reference" "#PWR01" (id 0) (at 50.8 119.38 0)
-      (effects (font (size 1.27 1.27)) hide)
-    )
-    (property "Value" "GND" (id 1) (at 50.8 118.11 0))
-    (property "Footprint" "" (id 2) (at 50.8 113.03 0)
-      (effects (font (size 1.27 1.27)) hide)
-    )
-    (property "Datasheet" "" (id 3) (at 50.8 113.03 0)
+  (symbol (lib_id "power:GND") (at 50.8 125.73 0) (unit 1)
+    (in_bom yes) (on_board yes) (fields_autoplaced)
+    (property "Reference" "#PWR01" (id 0) (at 50.8 132.08 0)
+      (effects (font (size 1.27 1.27)) hide)
+    )
+    (property "Value" "GND" (id 1) (at 50.8 130.81 0))
+    (property "Footprint" "" (id 2) (at 50.8 125.73 0)
+      (effects (font (size 1.27 1.27)) hide)
+    )
+    (property "Datasheet" "" (id 3) (at 50.8 125.73 0)
       (effects (font (size 1.27 1.27)) hide)
     )
@@
     )
     (path "/bcc2e053-f052-462b-8739-da56f79c71fe"
-      (reference "Q1") (unit 1) (value "2N3904") (footprint "Package_TO_SOT_THT:TO-92_Inline")
+      (reference "Q1") (unit 1) (value "2N3904") (footprint "Package_TO_SOT_THT:TO-92_Inline_Wide")
     )
     (path "/550a9c6f-df40-4a1c-9e90-c0271619fe3c"
@@
       (reference "R4") (unit 1) (value "220") (footprint "Resistor_THT:R_Axial_DIN0207_L6.3mm_D2.5mm_P10.16mm_Horizontal")
     )
-  )
+    (path "/2aa57eb1-108f-4543-9efb-ddacbac7b5fa"
+      (reference "SW1") (unit 1) (value "SW_SPDT") (footprint "Button_Switch_THT:SW_Slide_1P2T_CK_OS102011MS2Q")
+    )
+  )
